File: N12_TJA1103_KONG_KETI_EDUv2.kicad_pcb (KiCad board)
At the start: 2 copper layers, 33 x 57 mm, 65 parts, among them IC1 TJA1103AHN, J1 Conn_02x02_Odd_Even, J2 Conn_02x11_Odd_Even, J3 9-2304372-9, J4 E6S20A-40MT5-Z, Q1 FDN340P, Q2 BSS138, SW2 SW-DIP-ANGLED DS03-254-02BE, Y1 Crystal_GND24_Small

Commit message: fix: remove PCB shorts and dangling routing
Connections:
- FB1 pad 2: unconnected-(FB1-Pad2) -> VREGA_IN
- IC1 pad 16: unconnected-(IC1-VDDA_TRX-Pad16) -> VREGA_OUT
Routing:
- net Earth: track 42.7 -> 24.8 mm
- net /TX_EN: track 13.7 -> 5.42 mm
- net /DP+: track 16.5 -> 11.5 mm
- net /DN-: track 17.4 -> 13.7 mm
- net VDDD3V3: vias 10 -> 9
- net VDD3V3sw: vias 7 -> 6
