File: N12_TJA1103_KONG_KETI_EDUv2.kicad_sch (KiCad schematic)
At the start: 65 parts, among them IC1 TJA1103AHN, J1 Conn_02x02_Odd_Even, J2 Conn_02x11_Odd_Even, J3 9-2304372-9, J4 E6S20A-40MT5-Z, Q1 FDN340P, Q2 BSS138, SW2 SW-DIP-ANGLED DS03-254-02BE, Y1 Crystal_GND24_Small

Commit message: fix: resolve schematic footprint parity
Parts:
- FL1: footprint ACT45L_1 -> YK_Footprint_LIB:ACT45L_1
- IC1: footprint QFN50P600X600X100-37N-D -> YK_Footprint_LIB:QFN50P600X600X100-37N-D
- J4: footprint E6S20A:E6S20A40MT5Z -> YK_Footprint_LIB:E6S20A40MT5Z
Changed lines of the file:
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@@
 			)
 		)
-		(property "Footprint" "E6S20A:E6S20A40MT5Z"
+		(property "Footprint" "YK_Footprint_LIB:E6S20A40MT5Z"
 			(at 154.94 191.44 0)
 			(effects
@@
 			)
 		)
-		(property "Footprint" "ACT45L_1"
+		(property "Footprint" "YK_Footprint_LIB:ACT45L_1"
 			(at 158.75 116.51 0)
 			(effects
@@
 			)
 		)
-		(property "Footprint" "QFN50P600X600X100-37N-D"
+		(property "Footprint" "YK_Footprint_LIB:QFN50P600X600X100-37N-D"
 			(at 96.52 136.83 0)
 			(effects
